File: _saved_Rotherrie-Slomo-002.sch (KiCad schematic (older format))
At the start: 23 parts, among them U2 TL074

Commit message: Part associations made. 16pin connector reduced to 10 pin
Parts:
- R10, R11, R12, R13, R14, R15, R16, R5, R6, R7, R8, R9: footprint (none) -> Resistors_THT:R_Axial_DIN0207_L6.3mm_D2.5mm_P7.62mm_Horizontal
- RV1, RV2, RV3, RV4: footprint (none) -> Potentiometers:Potentiometer_Bourns_PTV09A-1_Horizontal
- U2: footprint (none) -> Housings_DIP:DIP-14_W7.62mm_Socket
Changed lines of the file:
@@
 F 0 "U2" H 3350 2550 50  0000 L CNN
 F 1 "TL074" H 3350 2150 50  0000 L CNN
-F 2 "" H 3300 2450 50  0001 C CNN
+F 2 "Housings_DIP:DIP-14_W7.62mm_Socket" H 3300 2450 50  0001 C CNN
 F 3 "" H 3400 2550 50  0001 C CNN
 	1    3350 2350
@@
 F 0 "R9" V 3230 1350 50  0000 C CNN
 F 1 "4.7k" V 3150 1350 50  0000 C CNN
-F 2 "" V 3080 1350 50  0001 C CNN
+F 2 "Resistors_THT:R_Axial_DIN0207_L6.3mm_D2.5mm_P7.62mm_Horizontal" V 3080 1350 50  0001 C CNN
 F 3 "" H 3150 1350 50  0001 C CNN
 	1    3150 1350
@@
 F 0 "R5" V 2080 1350 50  0000 C CNN
 F 1 "4.7k" V 2000 1350 50  0000 C CNN
-F 2 "" V 1930 1350 50  0001 C CNN
+F 2 "Resistors_THT:R_Axial_DIN0207_L6.3mm_D2.5mm_P7.62mm_Horizontal" V 1930 1350 50  0001 C CNN
 F 3 "" H 2000 1350 50  0001 C CNN
 	1    2000 1350
@@
 F 0 "R7" V 2430 2900 50  0000 C CNN
 F 1 "100k" V 2350 2900 50  0000 C CNN
-F 2 "" V 2280 2900 50  0001 C CNN
+F 2 "Resistors_THT:R_Axial_DIN0207_L6.3mm_D2.5mm_P7.62mm_Horizontal" V 2280 2900 50  0001 C CNN
 F 3 "" H 2350 2900 50  0001 C CNN
 	1    2350 2900
@@
 F 0 "RV1" V 2325 3300 50  0000 C CNN
 F 1 "500k" V 2400 3300 50  0000 C CNN
-F 2 "" H 2500 3300 50  0001 C CNN
+F 2 "Potentiometers:Potentiometer_Bourns_PTV09A-1_Horizontal" H 2500 3300 50  0001 C CNN
 F 3 "" H 2500 3300 50  0001 C CNN
 	1    2500 3300
@@
 F 0 "U2" H 6400 2550 50  0000 L CNN
 F 1 "TL074" H 6400 2150 50  0000 L CNN
-F 2 "" H 6350 2450 50  0001 C CNN
+F 2 "Housings_DIP:DIP-14_W7.62mm_Socket" H 6350 2450 50  0001 C CNN
 F 3 "" H 6450 2550 50  0001 C CNN
 	3    6400 2350
@@
 F 0 "R13" V 6280 1350 50  0000 C CNN
 F 1 "4.7k" V 6200 1350 50  0000 C CNN
-F 2 "" V 6130 1350 50  0001 C CNN
+F 2 "Resistors_THT:R_Axial_DIN0207_L6.3mm_D2.5mm_P7.62mm_Horizontal" V 6130 1350 50  0001 C CNN
 F 3 "" H 6200 1350 50  0001 C CNN
 	1    6200 1350
@@
 F 0 "R11" V 5130 1350 50  0000 C CNN
 F 1 "4.7k" V 5050 1350 50  0000 C CNN
-F 2 "" V 4980 1350 50  0001 C CNN
+F 2 "Resistors_THT:R_Axial_DIN0207_L6.3mm_D2.5mm_P7.62mm_Horizontal" V 4980 1350 50  0001 C CNN
 F 3 "" H 5050 1350 50  0001 C CNN
 	1    5050 1350
@@
 F 0 "R12" V 5480 2900 50  0000 C CNN
 F 1 "100k" V 5400 2900 50  0000 C CNN
-F 2 "" V 5330 2900 50  0001 C CNN
+F 2 "Resistors_THT:R_Axial_DIN0207_L6.3mm_D2.5mm_P7.62mm_Horizontal" V 5330 2900 50  0001 C CNN
 F 3 "" H 5400 2900 50  0001 C CNN
 	1    5400 2900
@@
 F 0 "RV3" V 5375 3300 50  0000 C CNN
 F 1 "500k" V 5450 3300 50  0000 C CNN
-F 2 "" H 5550 3300 50  0001 C CNN
+F 2 "Potentiometers:Potentiometer_Bourns_PTV09A-1_Horizontal" H 5550 3300 50  0001 C CNN
 F 3 "" H 5550 3300 50  0001 C CNN
 	1    5550 3300
@@
 F 0 "U2" H 9450 2550 50  0000 L CNN
 F 1 "TL074" H 9450 2150 50  0000 L CNN
-F 2 "" H 9400 2450 50  0001 C CNN
+F 2 "Housings_DIP:DIP-14_W7.62mm_Socket" H 9400 2450 50  0001 C CNN
 F 3 "" H 9500 2550 50  0001 C CNN
 	4    9450 2350
@@
 F 0 "R16" V 9330 1350 50  0000 C CNN
 F 1 "4.7k" V 9250 1350 50  0000 C CNN
-F 2 "" V 9180 1350 50  0001 C CNN
+F 2 "Resistors_THT:R_Axial_DIN0207_L6.3mm_D2.5mm_P7.62mm_Horizontal" V 9180 1350 50  0001 C CNN
 F 3 "" H 9250 1350 50  0001 C CNN
 	1    9250 1350
@@
 F 0 "R14" V 8180 1350 50  0000 C CNN
 F 1 "4.7k" V 8100 1350 50  0000 C CNN
-F 2 "" V 8030 1350 50  0001 C CNN
+F 2 "Resistors_THT:R_Axial_DIN0207_L6.3mm_D2.5mm_P7.62mm_Horizontal" V 8030 1350 50  0001 C CNN
 F 3 "" H 8100 1350 50  0001 C CNN
 	1    8100 1350
@@
 F 0 "R15" V 8530 2900 50  0000 C CNN
 F 1 "100k" V 8450 2900 50  0000 C CNN
-F 2 "" V 8380 2900 50  0001 C CNN
+F 2 "Resistors_THT:R_Axial_DIN0207_L6.3mm_D2.5mm_P7.62mm_Horizontal" V 8380 2900 50  0001 C CNN
 F 3 "" H 8450 2900 50  0001 C CNN
 	1    8450 2900
@@
 F 0 "RV4" V 8425 3300 50  0000 C CNN
 F 1 "500k" V 8500 3300 50  0000 C CNN
-F 2 "" H 8600 3300 50  0001 C CNN
+F 2 "Potentiometers:Potentiometer_Bourns_PTV09A-1_Horizontal" H 8600 3300 50  0001 C CNN
 F 3 "" H 8600 3300 50  0001 C CNN
 	1    8600 3300
@@
 F 0 "U2" H 3350 5500 50  0000 L CNN
 F 1 "TL074" H 3350 5100 50  0000 L CNN
-F 2 "" H 3300 5400 50  0001 C CNN
+F 2 "Housings_DIP:DIP-14_W7.62mm_Socket" H 3300 5400 50  0001 C CNN
 F 3 "" H 3400 5500 50  0001 C CNN
 	2    3350 5300
@@
 F 0 "R10" V 3230 4300 50  0000 C CNN
 F 1 "4.7k" V 3150 4300 50  0000 C CNN
-F 2 "" V 3080 4300 50  0001 C CNN
+F 2 "Resistors_THT:R_Axial_DIN0207_L6.3mm_D2.5mm_P7.62mm_Horizontal" V 3080 4300 50  0001 C CNN
 F 3 "" H 3150 4300 50  0001 C CNN
 	1    3150 4300
@@
 F 0 "R6" V 2080 4300 50  0000 C CNN
 F 1 "4.7k" V 2000 4300 50  0000 C CNN
-F 2 "" V 1930 4300 50  0001 C CNN
+F 2 "Resistors_THT:R_Axial_DIN0207_L6.3mm_D2.5mm_P7.62mm_Horizontal" V 1930 4300 50  0001 C CNN
 F 3 "" H 2000 4300 50  0001 C CNN
 	1    2000 4300
@@
 F 0 "R8" V 2430 5850 50  0000 C CNN
 F 1 "100k" V 2350 5850 50  0000 C CNN
-F 2 "" V 2280 5850 50  0001 C CNN
+F 2 "Resistors_THT:R_Axial_DIN0207_L6.3mm_D2.5mm_P7.62mm_Horizontal" V 2280 5850 50  0001 C CNN
 F 3 "" H 2350 5850 50  0001 C CNN
 	1    2350 5850
@@
 F 0 "RV2" V 2325 6250 50  0000 C CNN
 F 1 "500k" V 2400 6250 50  0000 C CNN
-F 2 "" H 2500 6250 50  0001 C CNN
+F 2 "Potentiometers:Potentiometer_Bourns_PTV09A-1_Horizontal" H 2500 6250 50  0001 C CNN
 F 3 "" H 2500 6250 50  0001 C CNN
 	1    2500 6250
