File: Rotherrie-Slomo.kicad_pcb (KiCad board)
At the start: 2 copper layers, 99.6 x 19.3 mm, 14 parts, among them J2 JACK_2P, J3 JACK_2P, J4 JACK_2P, J5 JACK_2P, J6 CONN_01X07, J7 CONN_01X07

Commit message: Finetuning controller board routing
Routing:
- net LED2: track 30.6 -> 28.9 mm
- net POT1: track 61.1 -> 59.4 mm
- net LED2R: track 27.7 -> 26.6 mm
- net WAVE2: track 48.2 -> 49.2 mm
- net LED4R: track 37.3 -> 36.7 mm
Changed lines of the file:
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@@
     (thickness 1.6)
     (drawings 4)
-    (tracks 127)
+    (tracks 120)
     (zones 0)
     (modules 14)
@@
   (segment (start 152.676001 61.838001) (end 153.576 62.738) (width 0.25) (layer F.Cu) (net 3))
   (segment (start 100.157001 62.057001) (end 141.436001 62.057001) (width 0.25) (layer F.Cu) (net 3))
-  (segment (start 114.808 52.832) (end 115.707999 53.731999) (width 0.25) (layer F.Cu) (net 5))
-  (segment (start 115.707999 53.731999) (end 127.479587 53.731999) (width 0.25) (layer F.Cu) (net 5))
-  (segment (start 127.479587 53.731999) (end 130.112649 51.098937) (width 0.25) (layer F.Cu) (net 5))
+  (segment (start 114.808 52.832) (end 116.830853 54.854853) (width 0.25) (layer F.Cu) (net 5))
+  (segment (start 116.830853 54.854853) (end 126.356733 54.854853) (width 0.25) (layer F.Cu) (net 5))
+  (segment (start 126.356733 54.854853) (end 130.112649 51.098937) (width 0.25) (layer F.Cu) (net 5))
   (segment (start 130.112649 51.098937) (end 132.0026 51.098937) (width 0.25) (layer F.Cu) (net 5))
+  (segment (start 142.358151 55.152574) (end 146.298134 51.212591) (width 0.25) (layer F.Cu) (net 5))
   (segment (start 132.0026 51.098937) (end 136.056237 55.152574) (width 0.25) (layer F.Cu) (net 5))
+  (segment (start 146.298134 51.212591) (end 146.598133 50.912592) (width 0.25) (layer F.Cu) (net 5))
   (segment (start 136.056237 55.152574) (end 142.358151 55.152574) (width 0.25) (layer F.Cu) (net 5))
-  (segment (start 142.358151 55.152574) (end 146.298134 51.212591) (width 0.25) (layer F.Cu) (net 5))
-  (segment (start 146.298134 51.212591) (end 146.598133 50.912592) (width 0.25) (layer F.Cu) (net 5))
   (segment (start 153.576 53.213) (end 153.576 50.358942) (width 0.25) (layer B.Cu) (net 5))
   (segment (start 153.576 50.358942) (end 151.788941 48.571883) (width 0.25) (layer B.Cu) (net 5))
@@
   (segment (start 86.36 61.202528) (end 89.662 64.504528) (width 0.25) (layer F.Cu) (net 11))
   (segment (start 89.662 64.504528) (end 89.662 64.516) (width 0.25) (layer F.Cu) (net 11))
-  (segment (start 107.599012 62.507012) (end 108.458 63.366) (width 0.25) (layer F.Cu) (net 12))
-  (segment (start 96.774 59.436) (end 99.845012 62.507012) (width 0.25) (layer F.Cu) (net 12))
-  (segment (start 94.488 55.372) (end 96.774 57.658) (width 0.25) (layer F.Cu) (net 12))
-  (segment (start 96.774 57.658) (end 96.774 59.436) (width 0.25) (layer F.Cu) (net 12))
-  (segment (start 91.186 55.372) (end 94.488 55.372) (width 0.25) (layer F.Cu) (net 12))
-  (segment (start 108.458 63.366) (end 108.458 64.516) (width 0.25) (layer F.Cu) (net 12))
-  (segment (start 99.845012 62.507012) (end 107.599012 62.507012) (width 0.25) (layer F.Cu) (net 12))
+  (segment (start 91.186 55.372) (end 92.71 55.372) (width 0.25) (layer F.Cu) (net 12))
+  (segment (start 106.949009 62.987374) (end 108.458 64.496365) (width 0.25) (layer F.Cu) (net 12))
+  (segment (start 92.71 55.372) (end 100.325374 62.987374) (width 0.25) (layer F.Cu) (net 12))
+  (segment (start 100.325374 62.987374) (end 106.949009 62.987374) (width 0.25) (layer F.Cu) (net 12))
+  (segment (start 108.458 64.496365) (end 108.458 64.516) (width 0.25) (layer F.Cu) (net 12))
   (segment (start 83.312 55.372) (end 91.186 55.372) (width 0.25) (layer B.Cu) (net 12) (status 10))
   (via (at 91.186 55.372) (size 0.6) (drill 0.4) (layers F.Cu B.Cu) (net 12))
-  (segment (start 91.186 56.388) (end 94.73057 56.388) (width 0.25) (layer F.Cu) (net 13))
-  (segment (start 94.73057 56.388) (end 96.24099 57.89842) (width 0.25) (layer F.Cu) (net 13))
-  (segment (start 96.24099 59.702234) (end 99.498795 62.960039) (width 0.25) (layer F.Cu) (net 13))
-  (segment (start 96.24099 57.89842) (end 96.24099 59.702234) (width 0.25) (layer F.Cu) (net 13))
-  (segment (start 99.498795 62.960039) (end 104.108039 62.960039) (width 0.25) (layer F.Cu) (net 13))
-  (segment (start 104.108039 62.960039) (end 105.664 64.516) (width 0.25) (layer F.Cu) (net 13))
+  (segment (start 91.186 56.388) (end 92.926756 56.388) (width 0.25) (layer F.Cu) (net 13))
+  (segment (start 92.926756 56.388) (end 101.054756 64.516) (width 0.25) (layer F.Cu) (net 13))
+  (segment (start 101.054756 64.516) (end 105.664 64.516) (width 0.25) (layer F.Cu) (net 13))
   (segment (start 105.664 64.516) (end 105.918 64.516) (width 0.25) (layer F.Cu) (net 13))
   (segment (start 83.312 57.912) (end 84.836 56.388) (width 0.25) (layer B.Cu) (net 13))
@@
   (segment (start 85.09 67.31) (end 138.684 67.31) (width 0.25) (layer F.Cu) (net 16))
   (segment (start 140.97 65.024) (end 140.97 64.516) (width 0.25) (layer F.Cu) (net 16) (status 30))
+  (segment (start 152.146 55.118) (end 152.146 52.062784) (width 0.25) (layer B.Cu) (net 17))
+  (segment (start 150.375216 50.292) (end 150.368 50.292) (width 0.25) (layer B.Cu) (net 17))
+  (segment (start 152.146 52.062784) (end 150.375216 50.292) (width 0.25) (layer B.Cu) (net 17))
   (segment (start 138.43 64.516) (end 138.43 64.262) (width 0.25) (layer F.Cu) (net 17))
   (segment (start 138.43 64.262) (end 139.7 62.992) (width 0.25) (layer F.Cu) (net 17))
-  (segment (start 151.384 50.292) (end 150.368 50.292) (width 0.25) (layer B.Cu) (net 17))
-  (segment (start 152.146 51.054) (end 151.384 50.292) (width 0.25) (layer B.Cu) (net 17))
-  (segment (start 152.146 55.118) (end 152.146 51.054) (width 0.25) (layer B.Cu) (net 17))
   (via (at 152.146 55.118) (size 0.6) (drill 0.4) (layers F.Cu B.Cu) (net 17))
   (segment (start 155.194 58.166) (end 152.146 55.118) (width 0.25) (layer F.Cu) (net 17))
@@
   (segment (start 138.43 64.516) (end 138.43 65.081998) (width 0.25) (layer B.Cu) (net 17) (status 30))
   (segment (start 98.552 55.332) (end 98.592 55.332) (width 0.25) (layer F.Cu) (net 18))
-  (segment (start 98.592 55.332) (end 101.328019 52.595981) (width 0.25) (layer F.Cu) (net 18))
+  (segment (start 98.592 55.332) (end 105.41 48.514) (width 0.25) (layer F.Cu) (net 18))
+  (segment (start 105.41 48.514) (end 145.542 48.514) (width 0.25) (layer F.Cu) (net 18))
+  (segment (start 145.542 48.514) (end 149.86 52.832) (width 0.25) (layer F.Cu) (net 18))
   (segment (start 149.86 52.832) (end 150.368 52.832) (width 0.25) (layer F.Cu) (net 18))
-  (segment (start 101.328019 52.595981) (end 101.328019 49.801981) (width 0.25) (layer F.Cu) (net 18))
-  (segment (start 145.542 48.514) (end 149.86 52.832) (width 0.25) (layer F.Cu) (net 18))
-  (segment (start 101.328019 49.801981) (end 102.616 48.514) (width 0.25) (layer F.Cu) (net 18))
-  (segment (start 102.616 48.514) (end 145.542 48.514) (width 0.25) (layer F.Cu) (net 18))
   (segment (start 98.552 57.832) (end 98.552 55.332) (width 0.25) (layer F.Cu) (net 18) (status 30))
   (segment (start 150.876 52.832) (end 150.368 52.832) (width 0.25) (layer B.Cu) (net 18) (status 30))
